File: hardware/sensors-minimal.kicad_sch (KiCad schematic)
At the start: 12 parts, among them U5 MMC5983MA, U6 MS560702BA03-50, U7 ADXL375BCCZ, U8 IIM-42653

Commit message: Removed bad GND connection to reserved pin on ADXL375 IMU; first error found in first batch
Connections:
- net GND: no longer U7.11 (RESERVED), U7.3 (RESERVED)
Changed lines of the file:
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@@
-	)
-	(junction
-		(at 233.68 137.16)
-		(diameter 0)
-		(color 0 0 0 0)
 	)
 	(junction
@@
 		(color 0 0 0 0)
 	)
-	(junction
-		(at 233.68 139.7)
-		(diameter 0)
-		(color 0 0 0 0)
-	)
 	(wire
 		(pts
@@
 	(wire
 		(pts
-			(xy 233.68 134.62) (xy 233.68 137.16)
+			(xy 233.68 134.62) (xy 233.68 139.7)
 		)
 		(stroke
@@
 	(wire
 		(pts
-			(xy 233.68 137.16) (xy 233.68 139.7)
-		)
-		(stroke
-			(width 0)
-			(type default)
-		)
-	)
-	(wire
-		(pts
 			(xy 29.21 156.21) (xy 30.48 156.21)
 		)
@@
 	(wire
 		(pts
-			(xy 227.33 139.7) (xy 233.68 139.7)
-		)
-		(stroke
-			(width 0)
-			(type default)
-		)
-	)
-	(wire
-		(pts
 			(xy 45.72 55.88) (xy 58.42 55.88)
 		)
@@
 		)
 		(stroke
-			(width 0)
-			(type default)
-		)
-	)
-	(wire
-		(pts
-			(xy 227.33 137.16) (xy 233.68 137.16)
-		)
-		(stroke
