File: hardware/active-drag-system.kicad_pcb (KiCad board)
At the start: 4 copper layers, 33 x 90 mm, 102 parts, among them J1 Conn_01x02_Pin, J2 Conn_01x02_Socket, J3 10118193-0001LF, J4 Conn_01x05_Pin, J5 Conn_01x02_Pin, J6 Conn_01x02_Pin, J7 Conn_01x03_Pin, J8 Conn_01x03_Pin, SW1 PTS815 SJM 250 SMTR LFS, U1 RP2040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

Commit message: sync
Parts:
- added TP10: nSLEEP, TestPoint:TestPoint_Pad_1.0x1.0mm, F.Cu at (157.9, 137.4)
- added TP11: DRVOFF, TestPoint:TestPoint_Pad_1.0x1.0mm, F.Cu at (153.3, 140.8)
- added TP12: BRAKE, TestPoint:TestPoint_Pad_1.0x1.0mm, B.Cu at (144.6, 125.9)
- added TP13: SPI_TX, TestPoint:TestPoint_Pad_1.0x1.0mm, F.Cu at (154.8, 128.0)
- added TP14: SPI_CSn, TestPoint:TestPoint_Pad_1.0x1.0mm, B.Cu at (147.6, 130.7)
- added TP15: SPI_SCK, TestPoint:TestPoint_Pad_1.0x1.0mm, F.Cu at (152.5, 130.2)
- added TP16: SPI_RX, TestPoint:TestPoint_Pad_1.0x1.0mm, F.Cu at (157.2, 128.0)
- added TP17: CLKIN, TestPoint:TestPoint_Pad_1.0x1.0mm, F.Cu at (155.0, 86.2)
- added TP18: MGINT, TestPoint:TestPoint_Pad_1.0x1.0mm, B.Cu at (159.2, 84.5)
- added TP19: MINT, TestPoint:TestPoint_Pad_1.0x1.0mm, B.Cu at (161.3, 71.5)
- added TP20: HGINT1, TestPoint:TestPoint_Pad_1.0x1.0mm, B.Cu at (157.4, 91.2)
- added TP21: HGINT2, TestPoint:TestPoint_Pad_1.0x1.0mm, F.Cu at (155.8, 95.8)
- added TP22: FGOUT, TestPoint:TestPoint_Pad_1.0x1.0mm, B.Cu at (133.5, 118.2)
- added TP9: nFAULT, TestPoint:TestPoint_Pad_1.0x1.0mm, F.Cu at (157.2, 140.8)
- J6: value Conn_01x02_Pin -> Conn_01x04_Pin; footprint Connector_PinHeader_2.54mm:PinHeader_1x02_P2.54mm_Vertical -> Connector_PinHeader_2.54mm:PinHeader_1x04_P2.54mm_Vertical
- moved J6 5.07 mm to (133.6, 113.6)
Connections:
- J6 pad 1: /MCU_RP2040/I2C1_SCL -> /+3V3
- J6 pad 2: /MCU_RP2040/I2C1_SDA -> GND
- U1 pad 7: unconnected-(U1-GPIO5-Pad7) -> /MCU_RP2040/FGOUT
- U1 pad 8: /MCU_RP2040/FGOUT -> unconnected-(U1-GPIO6-Pad8)
- U7 pad 11: GND -> unconnected-(U7-RESERVED-Pad11)
- U7 pad 3: GND -> unconnected-(U7-RESERVED-Pad3)
Routing:
- net /MCU_RP2040/SPI0_TX: track 54.7 -> 66.5 mm
- net /MAG: track 23.7 -> 30.7 mm, vias 2 -> 3
- net /MCU_RP2040/nSLEEP: track 57.5 -> 64.5 mm
- net /MCU_RP2040/SPI0_RX: track 53.5 -> 60.4 mm
- net /MCU_RP2040/nFAULT: track 59.6 -> 64.5 mm
- net /MCU_RP2040/SPI0_SCK: track 55.8 -> 60.0 mm
- net /MCU_RP2040/FGOUT: track 60.1 -> 62.1 mm
- net /HG2: track 10.3 -> 12.2 mm
- net /HG1: track 9.52 -> 11.3 mm, vias 0 -> 1
- net /MCU_RP2040/BRAKE: track 53.7 -> 55.5 mm
- net /MCU_RP2040/DRVOFF: track 60.0 -> 61.6 mm
- net /MG: track 12.6 -> 13.8 mm
- net /MCU_RP2040/CLKOUT: track 7.63 -> 8.66 mm
- net GND: track 236.4 -> 237.4 mm, vias 73 -> 74
- net /+3V3: track 21.8 -> 22.2 mm, vias 10 -> 14
Other:
- board text added: "Active Drag System: Rev 2 Designed by: Dawsyn Schraiber Kemper Brown Cian Capacci with help from Gabe Mills"
- board text added: "SWDIO GND SWCLK"
- board text added: "TX RX SDA SCL GND 3v3"
- board text removed: "Active Drag System: Rev 1 Designed by: Dawsyn Schraiber Kemper Brown Cian Capacci with help from Gabe Mills"
