File: hardware/mcu_rp2040.kicad_sch (KiCad schematic)
At the start: 30 parts, among them SW1 PTS815 SJM 250 SMTR LFS, U1 RP2040, U2 W25Q128JVSIQ, X1 ABM8AIG-12.000MHZ-12-2Z-T3

Commit message: Rev 2
Connections:
- net FGOUT: now also U1.7 (GPIO5); no longer U1.8 (GPIO6)
