File: hardware/motor_driver.kicad_sch (KiCad schematic)
At the start: 15 parts, among them U9 MCT8316Z0RRGFR

Commit message: Added digikey part numbers; usb trace width update
Parts:
- C36, C40: Digikey Part Number (none) -> 1276-1857-1-ND
- C37: Digikey Part Number (none) -> 490-10748-1-ND
- C38: Digikey Part Number (none) -> 490-4934-1-ND
- C39, C41: Digikey Part Number (none) -> 311-1868-1-ND
- C42: Digikey Part Number (none) -> 1276-7092-1-ND
- R17: Digikey Part Number (none) -> 13-RT0805BRD07164KLCT-ND
- R18: Digikey Part Number (none) -> P123795CT-ND
- R19, R21: Digikey Part Number (none) -> A102203CT-ND
- R20: Digikey Part Number (none) -> 13-RT0603BRD0722RLCT-ND
Changed lines of the file:
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@@
+			)
+		)
+		(property "Digikey Part Number" "A102203CT-ND"
+			(at 83.82 59.69 0)
+			(effects
+				(font
+					(size 1.27 1.27)
+				)
+				(hide yes)
 			)
 		)
@@
 			)
 		)
+		(property "Digikey Part Number" "P123795CT-ND"
+			(at 106.68 40.64 90)
+			(effects
+				(font
+					(size 1.27 1.27)
+				)
+				(hide yes)
+			)
+		)
 		(pin "2"
 		)
@@
 			)
 		)
+		(property "Digikey Part Number" "1276-1857-1-ND"
+			(at 152.4 41.91 0)
+			(effects
+				(font
+					(size 1.27 1.27)
+				)
+				(hide yes)
+			)
+		)
 		(pin "1"
 		)
@@
 			)
 		)
+		(property "Digikey Part Number" "490-4934-1-ND"
+			(at 124.46 45.72 90)
+			(effects
+				(font
+					(size 1.27 1.27)
+				)
+				(hide yes)
+			)
+		)
 		(pin "1"
 		)
@@
 					(size 0.635 0.635)
 				)
+			)
+		)
+		(property "Digikey Part Number" "1276-7092-1-ND"
+			(at 173.99 78.74 0)
+			(effects
+				(font
+					(size 1.27 1.27)
+				)
+				(hide yes)
 			)
 		)
@@
 			)
 		)
+		(property "Digikey Part Number" "13-RT0805BRD07164KLCT-ND"
+			(at 92.71 40.64 90)
+			(effects
+				(font
+					(size 1.27 1.27)
+				)
+				(hide yes)
+			)
+		)
 		(pin "2"
 		)
@@
 			)
 		)
+		(property "Digikey Part Number" "13-RT0603BRD0722RLCT-ND"
+			(at 163.83 74.93 90)
+			(effects
+				(font
+					(size 1.27 1.27)
+				)
+				(hide yes)
+			)
+		)
 		(pin "2"
 		)
@@
 			)
 		)
+		(property "Digikey Part Number" "311-1868-1-ND"
+			(at 173.99 60.96 0)
+			(effects
+				(font
+					(size 1.27 1.27)
+				)
+				(hide yes)
+			)
+		)
 		(pin "1"
 		)
@@
 			)
 		)
+		(property "Digikey Part Number" "1276-1857-1-ND"
+			(at 104.14 54.61 90)
+			(effects
+				(font
+					(size 1.27 1.27)
+				)
+				(hide yes)
+			)
+		)
 		(pin "1"
 		)
@@
 			)
 		)
+		(property "Digikey Part Number" "A102203CT-ND"
+			(at 78.74 76.2 0)
+			(effects
+				(font
+					(size 1.27 1.27)
+				)
+				(hide yes)
+			)
+		)
 		(pin "2"
 		)
@@
 			)
 		)
+		(property "Digikey Part Number" "490-10748-1-ND"
+			(at 161.29 41.91 0)
+			(effects
+				(font
+					(size 1.27 1.27)
+				)
+				(hide yes)
+			)
+		)
 		(pin "1"
 		)
@@
 			)
 		)
+		(property "Digikey Part Number" "311-1868-1-ND"
+			(at 134.62 48.26 90)
+			(effects
+				(font
+					(size 1.27 1.27)
+				)
+				(hide yes)
+			)
+		)

Commit message: Rev 2
Parts:
- added TP10: nSLEEP, TestPoint:TestPoint_Pad_1.0x1.0mm, symbol Connector:TestPoint
- added TP11: DRVOFF, TestPoint:TestPoint_Pad_1.0x1.0mm, symbol Connector:TestPoint
- added TP12: BRAKE, TestPoint:TestPoint_Pad_1.0x1.0mm, symbol Connector:TestPoint
- added TP13: SPI_TX, TestPoint:TestPoint_Pad_1.0x1.0mm, symbol Connector:TestPoint
- added TP14: SPI_CSn, TestPoint:TestPoint_Pad_1.0x1.0mm, symbol Connector:TestPoint
- added TP15: SPI_SCK, TestPoint:TestPoint_Pad_1.0x1.0mm, symbol Connector:TestPoint
- added TP16: SPI_RX, TestPoint:TestPoint_Pad_1.0x1.0mm, symbol Connector:TestPoint
- added TP22: FGOUT, TestPoint:TestPoint_Pad_1.0x1.0mm, symbol Connector:TestPoint
- added TP9: nFAULT, TestPoint:TestPoint_Pad_1.0x1.0mm, symbol Connector:TestPoint
Connections:
- net BRAKE: now also TP12.1
- net DRVOFF: now also TP11.1
- net FGOUT: now also TP22.1
- net SPI_CSn: now also TP14.1
- net SPI_RX: now also TP16.1
- net SPI_SCK: now also TP15.1
- net SPI_TX: now also TP13.1
- net nFAULT: now also TP9.1
- net nSLEEP: now also TP10.1
