File: hardware/power_regulation.kicad_sch (KiCad schematic)
At the start: 27 parts, among them U3 TPS51386RJNR, U4 LD39200PU33R

Commit message: Added digikey part numbers; usb trace width update
Parts:
- C16, C19: Digikey Part Number (none) -> 1276-1857-1-ND
- C17, C18, C26, C27: Digikey Part Number (none) -> 490-10748-1-ND
- C20, C21, C22, C23: Digikey Part Number (none) -> 1276-7092-1-ND
- C24: Digikey Part Number (none) -> 1292-1503-1-ND
- C25: Digikey Part Number (none) -> 311-1868-1-ND
- R10, R12, R13, R16: Digikey Part Number (none) -> P123795CT-ND
- R11: Digikey Part Number (none) -> A102216CT-ND
- R14, R15: Digikey Part Number (none) -> A102203CT-ND
Changed lines of the file:
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@@
+			)
+		)
+		(property "Digikey Part Number" "1276-7092-1-ND"
+			(at 204.47 49.53 0)
+			(effects
+				(font
+					(size 1.27 1.27)
+				)
+				(hide yes)
 			)
 		)
@@
 			)
 		)
+		(property "Digikey Part Number" "311-1868-1-ND"
+			(at 78.74 69.85 0)
+			(effects
+				(font
+					(size 1.27 1.27)
+				)
+				(hide yes)
+			)
+		)
 		(pin "1"
 		)
@@
 			)
 		)
+		(property "Digikey Part Number" "490-10748-1-ND"
+			(at 93.98 124.46 0)
+			(effects
+				(font
+					(size 1.27 1.27)
+				)
+				(hide yes)
+			)
+		)
 		(pin "1"
 		)
@@
 				)
 				(justify left)
+			)
+		)
+		(property "Digikey Part Number" "490-10748-1-ND"
+			(at 171.45 124.46 0)
+			(effects
+				(font
+					(size 1.27 1.27)
+				)
+				(hide yes)
 			)
 		)
@@
 			)
 		)
+		(property "Digikey Part Number" "P123795CT-ND"
+			(at 78.74 59.69 0)
+			(effects
+				(font
+					(size 1.27 1.27)
+				)
+				(hide yes)
+			)
+		)
 		(pin "2"
 		)
@@
 			)
 		)
+		(property "Digikey Part Number" "P123795CT-ND"
+			(at 105.41 124.46 0)
+			(effects
+				(font
+					(size 1.27 1.27)
+				)
+				(hide yes)
+			)
+		)
 		(pin "2"
 		)
@@
 			)
 		)
+		(property "Digikey Part Number" "1276-1857-1-ND"
+			(at 151.13 40.64 90)
+			(effects
+				(font
+					(size 1.27 1.27)
+				)
+				(hide yes)
+			)
+		)
 		(pin "1"
 		)
@@
 			)
 		)
+		(property "Digikey Part Number" "A102203CT-ND"
+			(at 149.86 64.77 0)
+			(effects
+				(font
+					(size 1.27 1.27)
+				)
+				(hide yes)
+			)
+		)
 		(pin "2"
 		)
@@
 				)
 				(justify left)
+			)
+		)
+		(property "Digikey Part Number" "490-10748-1-ND"
+			(at 49.53 44.45 0)
+			(effects
+				(font
+					(size 1.27 1.27)
+				)
+				(hide yes)
 			)
 		)
@@
 			)
 		)
+		(property "Digikey Part Number" "P123795CT-ND"
+			(at 68.58 58.42 0)
+			(effects
+				(font
+					(size 1.27 1.27)
+				)
+				(hide yes)
+			)
+		)
 		(pin "2"
 		)
@@
 			)
 		)
+		(property "Digikey Part Number" "1276-7092-1-ND"
+			(at 227.33 49.53 0)
+			(effects
+				(font
+					(size 1.27 1.27)
+				)
+				(hide yes)
+			)
+		)
 		(pin "2"
 		)
@@
 			)
 		)
+		(property "Digikey Part Number" "490-10748-1-ND"
+			(at 38.1 44.45 0)
+			(effects
+				(font
+					(size 1.27 1.27)
+				)
+				(hide yes)
+			)
+		)
 		(pin "1"
 		)
@@
 					(size 1.27 1.27)
 				)
+			)
+		)
+		(property "Digikey Part Number" "A102203CT-ND"
+			(at 149.86 74.93 0)
+			(effects
+				(font
+					(size 1.27 1.27)
+				)
+				(hide yes)
 			)
 		)
@@
 			)
 		)
+		(property "Digikey Part Number" "1292-1503-1-ND"
+			(at 176.53 58.42 90)
+			(effects
+				(font
+					(size 1.27 1.27)
+				)
+				(hide yes)
+			)
+		)
 		(pin "1"
 		)
@@
 		)
 		(property "LCSC" "C25755"
+			(at 162.56 54.61 90)
+			(effects
+				(font
+					(size 1.27 1.27)
+				)
+				(hide yes)
+			)
+		)
+		(property "Digikey Part Number" "A102216CT-ND"
 			(at 162.56 54.61 90)
 			(effects
@@
 			)
 		)
+		(property "Digikey Part Number" "1276-7092-1-ND"
+			(at 191.77 49.53 0)
+			(effects
+				(font
+					(size 1.27 1.27)
+				)
+				(hide yes)
+			)
+		)
 		(pin "2"
 		)
@@
 			)
 		)
+		(property "Digikey Part Number" "1276-1857-1-ND"
+			(at 60.96 44.45 0)
+			(effects
+				(font
+					(size 1.27 1.27)
+				)
+				(hide yes)
+			)
+		)
 		(pin "1"
 		)
@@
 					(size 0.635 0.635)
 				)
+			)
+		)
+		(property "Digikey Part Number" "1276-7092-1-ND"
+			(at 215.9 49.53 0)
+			(effects
+				(font
+					(size 1.27 1.27)
+				)
+				(hide yes)
 			)
 		)
@@
 			)
 		)
+		(property "Digikey Part Number" "P123795CT-ND"
+			(at 85.09 46.99 0)
+			(effects
+				(font
+					(size 1.27 1.27)
+				)
+				(hide yes)
+			)
+		)

Commit message: Rev 2
Changed lines of the file:
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@@
 (kicad_sch
-	(version 20231120)
+	(version 20250114)
 	(generator "eeschema")
-	(generator_version "8.0")
+	(generator_version "9.0")
 	(paper "USLetter")
 	(junction
@@
 			"yy/J7zz3Yt5aOp+/ztzriMoFAACfSDgAAAAAAABAa1wo7bv8e6lYxLldIexiMWYhdb9SOhgAAAAA"
 			"AAAA4N2Fue6VcAgOAKAu/x+BQhr0wIjOiwAAAA5lWElmTU0AKgAAAAgAAAAAAAAA0lOTAAAAAElF"
-			"TkSuQmCC"
+			"TkSuQmCCAEUAAABCAAAAQQAAAEQAAABCAAAAMAAAADEAAAA2AAAASQAAAEQAAABBAAAAQQAAAEEA"
+			"AABBAAAAQQAAAEEAAABEAAAAKwAAAFQAAABuAAAAQQAAAEEAAABBAAAAQQAAAEEAAABBAAAAOAAA"
+			"AEEAAAA3AAAANwAAADIAAABPAAAAQgAAAHoAAAA5AAAAZwAAADQAAABBAAAAZwAAAEMAAABNAAAA"
+			"UgAAAEgAAABRAAAAQQAAAEEAAABBAAAAQQAAAEEAAABBAAAAOAAAAEIAAABmAAAAQgAAAEEAAABR"
+			"AAAAQQAAAEEAAABBAAAATQAAAEEAAABiAAAAdAAAAFYAAABLAAAAdgAAAFEAAABtAAAAdwAAAEEA"
+			"AABBAAAASQAAAHoAAABQAAAAZAAAAFMAAAB2AAAAMQAAAFMAAAB5AAAAdAAAADEAAABuAAAAagAA"
+			"ADAAAABFAAAAQQAAAEEAAABBAAAAQQAAAEEAAABJAAAAQgAAAGMAAABnAAAAZwAAAE0AAABBAAAA"
+			"QQAAAEEAAABDAAAAQQAAAE4AAAAyAAAAaQAAAGwAAABYAAAAawAAAGIAAABFAAAATgAAAG4AAABz"
+			"AAAASAAAAEEAAABNAAAAQwAAAEoAAABYAAAARQAAAFQAAABFAAAAZwAAACsAAABnAAAAQQAAAEEA"
+			"AABBAAAAQQAAAEEAAABBAAAARwAAAEQAAABhAAAAQgAAAEEAAABjAAAAQQAAAEEAAABBAAAAQQAA"
+			"AEEAAAByAAAANwAAAFMAAABQAAAARAAAAFIAAAA0AAAAaQAAAFkAAABwAAAAWQAAADgAAABCAAAA"
+			"UQAAAEQAAABnAAAAbAAAAEMAAAA0AAAAaQAAADQAAABzAAAAdgAAACsAAAB1AAAAdwAAADgAAABB"
+			"AAAAQQAAAEEAAABBAAAAQQAAAEEAAABCAAAATQAAAGsAAABPAAAAQQAAAEEAAABBAAAAQQAAAEEA"
+			"AABCAAAANAAAAEIAAABiAAAARQAAAEIAAABBAAAARAAAAEEAAAB4AAAAaQAAADkAAABoAAAAZAAA"
+			"AE8AAABoAAAAQQAAAGQAAABBAAAAQQAAAEEAAABBAAAAQQAAAEEAAABCAAAATQAAAGsAAABPAAAA"
+			"QQAAAEEAAABBAAAAQQAAAEEAAABBAAAANAAAAEUAAABDAAAAdAAAADEAAABIAAAAbQAAAEkAAABE"
+			"AAAAUQAAAEMAAABBAAAANgAAAFoAAABuAAAARgAAAEwAAABqAAAAcAAAAFkAAABaAAAAdwAAADgA"
+			"AABCAAAAQQAAAEEAAABBAAAAQQAAAEEAAABPAAAAQwAAADgAAABCAAAAQQAAAGMAAABBAAAAQQAA"
+			"AEEAAABvAAAANgAAAGUAAAB3AAAAZwAAAEEAAABBAAAAQQAAAEEAAABBAAAAQQAAAE8AAAA4AAAA"
+			"agAAAE8AAABBAAAAQQAAAEEAAABBAAAAQQAAAEEAAABtAAAAVAAAAFcAAAB3AAAAQQAAAEEAAABI"
+			"AAAAQQAAAFMAAABzAAAANAAAAGoAAAA0AAAAMwAAAEUAAABxAAAAOQAAAHoAAABSAAAANAAAAEMA"
+			"AABBAAAAQQAAAEEAAABBAAAAQQAAAE0AAABEAAAAYgAAAEMAAABRAAAANAAAAEEAAABBAAAAQQAA"
+			"AEMAAABBAAAAeQAAAFcAAABxAAAAbAAAAGwAAABoAAAAQQAAAGIAAABBAAAAQQAAAEMAAABjAAAA"
+			"MAAAAHMAAABkAAAAVwAAADYAAABzAAAATQAAACsAAAA4AAAAZwAAAFEAAABBAAAAQQAAAEEAAABB"
+			"AAAAQQAAAFkAAABHAAAAQQAAAEUAAABCAAAAdwAAAEEAAABBAAAAQQAAAE0AAABBAAAAawAAAHQA"
+			"AABWAAAASQAAAHYAAABJAAAAKwAAAEoAAABMAAAAaQAAAEEAAAAwAAAAQQAAAEEAAABFAAAANQAA"
+			"AHQAAABHAAAAUgAAAEcAAABQAAAAKwAAACsAAAA5AAAAZgAAAEEAAABBAAAAQQAAAEEAAABBAAAA"
+			"QQAAAEEAAABNAAAAaQAAAE8AAABBAAAAQQAAAEEAAABBAAAAQQAAAEEAAABtAAAASgAAAHoAAAA5"
+			"AAAAagAAADkAAAAwAAAAZQAAAEkAAABtAAAASwAAAFcAAABQAAAAQQAAAFUAAABBAAAAWQAAAEMA"
+			"AABwAAAAbQAAAEUAAABmAAAASAAAAHYAAABWAAAAdQAAAG8AAABtAAAAZQAAAHcAAABnAAAAQQAA"
+			"AEEAAABBAAAAQQAAAEEAAABBAAAASQAAAGMAAABUAAAASAAAAEEAAABBAAAAQQAAAEEAAABBAAAA"
+			"QwAAAFQAAABJAAAAagAAAFkAAABBAAAAQQAAAEUAAABqAAAAMQAAAGEAAAB5AAAAdgAAADEAAABy"
+			"AAAAcAAAAFUAAAA2AAAAegAAAHgAAAA0AAAAQwAAAEEAAABBAAAAQQAAAEEAAABBAAAATQAAAEQA"
+			"AABMAAAAQgAAAEEAAABjAAAAQQAAAEEAAABBAAAARAAAAEEAAABaAAAATAAAAFIAAABTAAAAcgAA"
+			"ADAAAABKAAAAcwAAAEEAAABBAAAAQwAAAFEAAAA3AAAAVQAAAE4AAABFAAAAZgAAAE4AAABtAAAA"
+			"SAAAAG8AAABBAAAAQQAAAEEAAABBAAAAQQAAAEEAAABBAAAAOQAAAEoAAABqAAAAZwAAAEEAAABB"
+			"AAAAQQ=="
 		)
 	)
@@
 		(shape input)
 		(at 39.37 35.56 0)
-		(fields_autoplaced yes)
 		(effects
 			(font
@@
 		(shape output)
 		(at 228.6 38.1 0)
-		(fields_autoplaced yes)
 		(effects
 			(font
@@
 		(shape output)
 		(at 82.55 104.14 180)
-		(fields_autoplaced yes)
 		(effects
 			(font
@@
 		(shape output)
 		(at 171.45 107.95 0)
-		(fields_autoplaced yes)
 		(effects
 			(font
@@
 		(shape input)
 		(at 95.25 104.14 0)
-		(fields_autoplaced yes)
 		(effects
 			(font
