File: hardware/sensors.kicad_sch (KiCad schematic)
At the start: 12 parts, among them U5 MMC5983MA, U6 MS560702BA03-50, U7 ADXL375BCCZ, U8 IIM-42653

Commit message: Rev 2
Parts:
- added TP17: CLKIN, TestPoint:TestPoint_Pad_1.0x1.0mm, symbol Connector:TestPoint
- added TP18: MGINT, TestPoint:TestPoint_Pad_1.0x1.0mm, symbol Connector:TestPoint
- added TP19: MINT, TestPoint:TestPoint_Pad_1.0x1.0mm, symbol Connector:TestPoint
- added TP20: HGINT1, TestPoint:TestPoint_Pad_1.0x1.0mm, symbol Connector:TestPoint
- added TP21: HGINT2, TestPoint:TestPoint_Pad_1.0x1.0mm, symbol Connector:TestPoint
Connections:
- net CLKIN: now also TP17.1
- net HIGHG_INT1: now also TP20.1
- net HIGHG_INT2: now also TP21.1
- net MAG_INT: now also TP19.1
- net MIDG_INT: now also TP18.1
